File: motores.kicad_sch (KiCad schematic)
At the start: 7 parts

Commit message: fix: modificado saídas do arduino
Parts:
- U1, U2: renamed from U?; footprint (none) -> Connector_PinSocket_2.54mm:PinSocket_2x04_P2.54mm_Vertical
- gave numbers to parts that had none: 5

Commit message: fix: mudanca dos pinos de alimentacao
Connections:
- net 5V_Ard renamed 5V_Sen
Changed lines of the file:
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@@
     (effects (font (size 1.27 1.27)) (justify left bottom))
   )
-  (global_label "5V_Ard" (shape bidirectional) (at 26.67 39.37 90) (fields_autoplaced)
+  (global_label "5V_Sen" (shape bidirectional) (at 26.67 39.37 90) (fields_autoplaced)
     (effects (font (size 1.27 1.27)) (justify left))
-    (property "Intersheetrefs" "${INTERSHEET_REFS}" (at 26.67 28.984 90)
+    (property "Intersheetrefs" "${INTERSHEET_REFS}" (at 26.67 28.5607 90)
       (effects (font (size 1.27 1.27)) (justify left))
     )
@@
     )
   )
-  (global_label "5V_Ard" (shape bidirectional) (at 86.36 39.37 90) (fields_autoplaced)
+  (global_label "5V_Sen" (shape bidirectional) (at 86.36 39.37 90) (fields_autoplaced)
     (effects (font (size 1.27 1.27)) (justify left))
-    (property "Intersheetrefs" "${INTERSHEET_REFS}" (at 86.36 28.984 90)
+    (property "Intersheetrefs" "${INTERSHEET_REFS}" (at 86.36 28.5607 90)
       (effects (font (size 1.27 1.27)) (justify left))
     )
