File: sensores.kicad_sch (KiCad schematic)
At the start: 8 parts

Commit message: fix: modificado saídas do arduino
Parts:
- U10, U11: renamed from U?; footprint (none) -> Connector_PinHeader_2.54mm:PinHeader_1x03_P2.54mm_Vertical
- U12: renamed from U?; footprint (none) -> Connector_FFC-FPC:Molex_200528-0060_1x06-1MP_P1.00mm_Horizontal
- U5, U6, U7: renamed from U?; footprint (none) -> Connector_PinSocket_2.54mm:PinSocket_1x04_P2.54mm_Vertical
- U8, U9: renamed from U?; footprint (none) -> TerminalBlock_Phoenix:TerminalBlock_Phoenix_MKDS-1,5-4_1x04_P5.00mm_Horizontal

Commit message: fix: mudanca dos pinos de alimentacao
Connections:
- net 5V_Ard: now also U8. (SW); no longer U10. (VCC), U11. (VCC), U12. (XDA)
- net 5V_Sen: now also U10. (VCC), U11. (VCC), U12. (XDA), U5. (VCC), U6. (VCC), U7. (VCC); no longer U8. (SW)
- removed net +5V: U5. (VCC), U6. (VCC), U7. (VCC)
Changed lines of the file:
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@@
     (rev "2023-09-04")
-  )
-  (junction (at 30.48 39.37) (diameter 0) (color 0 0 0 0)
   )
   (junction (at 30.48 63.5) (diameter 0) (color 0 0 0 0)
@@
   )
   (wire (pts (xy 43.18 87.63) (xy 43.18 86.36))
-    (stroke (width 0) (type default))
-  )
-  (wire (pts (xy 30.48 35.56) (xy 30.48 39.37))
     (stroke (width 0) (type default))
   )
@@
     (effects (font (size 1.27 1.27)) (justify left bottom))
   )
-  (global_label "5V_Ard" (shape bidirectional) (at 106.68 36.83 90) (fields_autoplaced)
+  (global_label "5V_Sen" (shape bidirectional) (at 106.68 36.83 90) (fields_autoplaced)
     (effects (font (size 1.27 1.27)) (justify left))
-    (property "Intersheetrefs" "${INTERSHEET_REFS}" (at 106.68 26.444 90)
+    (property "Intersheetrefs" "${INTERSHEET_REFS}" (at 106.68 26.0207 90)
       (effects (font (size 1.27 1.27)) (justify left))
     )
   )
-  (global_label "5V_Ard" (shape bidirectional) (at 214.63 35.56 90) (fields_autoplaced)
+  (global_label "5V_Sen" (shape bidirectional) (at 214.63 35.56 90) (fields_autoplaced)
     (effects (font (size 1.27 1.27)) (justify left))
-    (property "Intersheetrefs" "${INTERSHEET_REFS}" (at 214.63 25.174 90)
+    (property "Intersheetrefs" "${INTERSHEET_REFS}" (at 214.63 24.7507 90)
       (effects (font (size 1.27 1.27)) (justify left))
     )
@@
     )
   )
-  (global_label "5V_Ard" (shape bidirectional) (at 149.86 36.83 90) (fields_autoplaced)
+  (global_label "5V_Sen" (shape bidirectional) (at 149.86 36.83 90) (fields_autoplaced)
     (effects (font (size 1.27 1.27)) (justify left))
-    (property "Intersheetrefs" "${INTERSHEET_REFS}" (at 149.86 26.444 90)
+    (property "Intersheetrefs" "${INTERSHEET_REFS}" (at 149.86 26.0207 90)
       (effects (font (size 1.27 1.27)) (justify left))
     )
@@
     )
   )
+  (global_label "5V_Sen" (shape bidirectional) (at 30.48 87.63 270) (fields_autoplaced)
+    (effects (font (size 1.27 1.27)) (justify right))
+    (property "Intersheetrefs" "${INTERSHEET_REFS}" (at 30.48 98.4393 90)
+      (effects (font (size 1.27 1.27)) (justify right))
+    )
+  )
   (global_label "IR1" (shape bidirectional) (at 96.52 45.72 180) (fields_autoplaced)
     (effects (font (size 1.27 1.27)) (justify right))
@@
     )
   )
-  (global_label "5V_Sen" (shape bidirectional) (at 46.99 132.08 180) (fields_autoplaced)
+  (global_label "5V_Ard" (shape bidirectional) (at 46.99 132.08 180) (fields_autoplaced)
     (effects (font (size 1.27 1.27)) (justify right))
-    (property "Intersheetrefs" "${INTERSHEET_REFS}" (at 36.1807 132.08 0)
+    (property "Intersheetrefs" "${INTERSHEET_REFS}" (at 36.604 132.08 0)
       (effects (font (size 1.27 1.27)) (justify right))
     )
@@
         )
       )
-    )
-  )
-  (symbol (lib_id "power:+5V") (at 30.48 35.56 0) (unit 1)
-    (in_bom yes) (on_board yes) (dnp no) (fields_autoplaced)
-    (property "Reference" "#PWR018" (at 30.48 39.37 0)
-      (effects (font (size 1.27 1.27)) hide)
-    )
-    (property "Value" "+5V" (at 30.48 30.48 0)
-      (effects (font (size 1.27 1.27)))
-    )
-    (property "Footprint" "" (at 30.48 35.56 0)
-      (effects (font (size 1.27 1.27)) hide)
-    )
-    (property "Datasheet" "" (at 30.48 35.56 0)
-      (effects (font (size 1.27 1.27)) hide)
-    )
-    (pin "1")
-    (instances
-      (project "esquemaEletricoCarro"
-        (path "/e63e39d7-6ac0-4ffd-8aa3-1841a4541b55/ef1da815-5ae9-4f7a-859c-d7960e6acc1e"
-          (reference "#PWR018") (unit 1)
-        )
-      )

Commit message: fix: mudanca das conexoes
Changed lines of the file:
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@@
     )
   )
-  (global_label "IR1" (shape bidirectional) (at 96.52 45.72 180) (fields_autoplaced)
+  (global_label "IR1" (shape bidirectional) (at 96.52 43.18 180) (fields_autoplaced)
     (effects (font (size 1.27 1.27)) (justify right))
-    (property "Intersheetrefs" "${INTERSHEET_REFS}" (at 89.3392 45.72 0)
+    (property "Intersheetrefs" "${INTERSHEET_REFS}" (at 89.3392 43.18 0)
       (effects (font (size 1.27 1.27)) (justify right))
     )
@@
     )
   )
-  (global_label "IR2" (shape bidirectional) (at 139.7 45.72 180) (fields_autoplaced)
+  (global_label "IR2" (shape bidirectional) (at 139.7 43.18 180) (fields_autoplaced)
     (effects (font (size 1.27 1.27)) (justify right))
-    (property "Intersheetrefs" "${INTERSHEET_REFS}" (at 132.5192 45.72 0)
+    (property "Intersheetrefs" "${INTERSHEET_REFS}" (at 132.5192 43.18 0)
       (effects (font (size 1.27 1.27)) (justify right))
     )

Commit message: fix: esquematico atualizado
Parts:
- removed U10, U11: TCRT5000, Connector_PinHeader_2.54mm:PinHeader_1x03_P2.54mm_Vertical, symbol Customizados:TCRT5000
- added SC1, SC2: Solar_Cell, symbol Device:Solar_Cell
- added U?: Controladora 12V Placa Solar, symbol Customizados:Controladora_12V_Placa_Solar
- added U? (x2): Sensor de tensão, symbol Customizados:Sensor_de_tensão
Connections:
- net 5V_Ard: now also U?. (VCC), U?. (VCC)
- net Earth: now also U?. (PlaSol-), U?. (VCC), U?. (VCC)
- new net: SC1.1 (+), SC2.1 (+), U?. (PlaSol-), U?. (VCC)
- new net: SC1.2 (-), SC2.2 (-), U?. (PlaSol-), U?. (VCC)
- new net 12V_Mot: U?. (PlaSol-), U?. (VCC)
- new net U_Mot: U?. (VCC)
- new net U_PlaSol: U?. (VCC)
Other:
- moved on the sheet: U12
